Commit message: Apply SyncRobot create_robot changes

File: create_description/urdf/create_base.urdf.xacro (robot description, xacro)
@@ -197,4 +197,32 @@
     </inertial>
     </link>
+    <joint name="laser_joint" type="fixed">
+      <axis xyz="0 1 0" />
+      <origin xyz="0.10 0 0.08" rpy="0 0 ${PI}" />
+      <parent link="base_link" />
+      <child link="laser" />
+    </joint>
+    <link name="laser">
+    <inertial>
+      <mass value="0.190" />
+      <origin xyz="0 0 0" rpy="0 0 0" />
+      <inertia ixx="0.000095" ixy="0" ixz="0" iyy="0.000095" iyz="0" izz="0.000054" />
+    </inertial>
+    <visual>
+      <origin xyz="0 0 0" rpy="0 0 0" />
+      <geometry>
+        <cylinder radius="0.0254" length="0.04" />
+      </geometry>
+      <material name="lidar_black">
+        <color rgba="0.1 0.1 0.1 1.0" />
+      </material>
+    </visual>
+    <collision>
+      <origin xyz="0 0 0" rpy="0 0 0" />
+      <geometry>
+        <cylinder radius="0.0254" length="0.04" />
+      </geometry>
+    </collision>
+    </link>
     <!-- Simulation sensors -->
     <xacro:sim_create_base/>
